File: KiCad/LISA_to_FPGA.sch (KiCad schematic (older format))
At the start: 14 parts, among them J1 Conn_01x02, J2 Conn_01x02, J3 Conn_01x40, U1 LM1117-3.3, U2 74LVC245A, U3 74LVC245A, U5 LISA

Commit message: more place and route
Parts:
- removed J1, J2: Conn_01x02, Connector_PinHeader_2.54mm:PinHeader_1x02_P2.54mm_Horizontal, symbol Connector_Generic:Conn_01x02
- added J1: Conn_01x03, Connector_PinHeader_2.54mm:PinHeader_1x03_P2.54mm_Horizontal, symbol Connector_Generic:Conn_01x03
- added U3, U5: 74LVC245A, Package_SO:TSSOP-20_4.4x6.5mm_P0.65mm, symbol LISA_to_FPGA:74LVC245A
- C3, C4, C5: footprint Capacitor_SMD:C_0805_2012Metric_Pad1.15x1.40mm_HandSolder -> Capacitor_SMD:C_0603_1608Metric_Pad1.08x0.95mm_HandSolder
- C6: footprint Capacitor_SMD:C_0805_2012Metric_Pad1.18x1.45mm_HandSolder -> Capacitor_SMD:C_0603_1608Metric_Pad1.08x0.95mm_HandSolder
- U6: renamed from U5; footprint Package_LCC:PLCC-84_THT-Socket -> LISA_to_FPGA:PLCC-84_THT-Socket-HAT
- renumbered J3 to J2, U3 to U2, U2 to U4
Connections:
- net 3V3: now also U3.1 (DIR), U3.20 (VCC), U5.1 (DIR), U5.20 (VCC)
- net B0: now also U3.5 (A3)
- net B0_3V3: now also U3.15 (B3)
- net B1: now also U3.6 (A4)
- net B1_3V3: now also U3.14 (B4)
- net B2: now also U3.7 (A5)
- net B2_3V3: now also U3.13 (B5)
- net B3: now also U3.8 (A6)
- net B3_3V3: now also U3.12 (B6)
- net B4: now also U3.9 (A7); no longer U2.2 (A0)
- net B4_3V3: now also U3.11 (B7); no longer U2.18 (B0)
- net B5: now also U2.2 (A0); no longer U2.3 (A1)
- net B5_3V3: now also U2.18 (B0); no longer U2.17 (B1)
- net B6: now also U2.3 (A1); no longer U2.4 (A2)
- net B6_3V3: now also U2.17 (B1); no longer U2.16 (B2)
- net B7: now also U2.4 (A2); no longer U2.5 (A3)
- net B7_3V3: now also U2.16 (B2); no longer U2.15 (B3)
- net C14OUT: now also U2.9 (A7); no longer R1.2
- net CSYNC: now also U2.5 (A3), J1.1 (Pin_1); no longer U2.6 (A4)
- net CSYNC_3V3: now also U2.15 (B3); no longer U2.14 (B4)
- net G0: now also U4.5 (A3)
- net G0_3V3: now also U4.15 (B3)
- net G1: now also U4.6 (A4)
- net G1_3V3: now also U4.14 (B4)
- net G2: now also U4.7 (A5)
- net G2_3V3: now also U4.13 (B5)
- net G3: now also U4.8 (A6)
- net G3_3V3: now also U4.12 (B6)
- net G4: now also U4.9 (A7); no longer U4.6 (A4)
- net G4_3V3: now also U4.11 (B7); no longer U4.14 (B4)
- net G5: now also U3.2 (A0); no longer U4.7 (A5)
- net G5_3V3: now also U3.18 (B0); no longer U4.13 (B5)
- net G6: now also U3.3 (A1); no longer U4.8 (A6)
- net G6_3V3: now also U3.17 (B1); no longer U4.12 (B6)
- net G7: now also U3.4 (A2); no longer U4.9 (A7)
- net G7_3V3: now also U3.16 (B2); no longer U4.11 (B7)
- net GND: now also U3.10 (GND), U3.19 (~OE), U5.10 (GND), U5.19 (~OE), U5.2 (A0), U5.3 (A1), U5.4 (A2)
- net HSYNC: now also U2.7 (A5), J1.2 (Pin_2); no longer U2.8 (A6)
- net HSYNC_3V3: now also U2.13 (B5); no longer U2.12 (B6)
- net PIXELSW: now also U2.6 (A4); no longer U2.7 (A5)
- net PIXELSW_3V3: now also U2.14 (B4); no longer U2.13 (B5)
- net R0: now also U5.5 (A3)
- net R0_3V3: now also U5.15 (B3)
- net R1: now also U5.6 (A4)
- net R1_3V3: now also U5.14 (B4)
- net R2: now also U5.7 (A5)
- net R2_3V3: now also U5.13 (B5)
- net R3: now also U5.8 (A6)
- net R3_3V3: now also U5.12 (B6)
- net R4: now also U5.9 (A7); no longer U4.2 (A0)
- net R4_3V3: now also U5.11 (B7); no longer U4.18 (B0)
- net R5: now also U4.2 (A0); no longer U4.3 (A1)
- net R5_3V3: now also U4.18 (B0); no longer U4.17 (B1)
- net R6: now also U4.3 (A1); no longer U4.4 (A2)
- net R6_3V3: now also U4.17 (B1); no longer U4.16 (B2)
- net R7: now also U4.4 (A2); no longer U4.5 (A3)
- net R7_3V3: now also U4.16 (B2); no longer U4.15 (B3)
- net VSYNC: now also U2.8 (A6), J1.3 (Pin_3); no longer U2.9 (A7)
- net VSYNC_3V3: now also U2.12 (B6); no longer U2.11 (B7)
- new net C14OUT_3V3: R1.2, U2.11 (B7)
- no-connect marks 59 -> 61
Other:
- moved on the sheet: R1, U2, U4
