File: A1200/KiCad/LISA_to_FPGA.sch (KiCad schematic (older format))
At the start: 15 parts, among them J1 Conn_01x03, J2 Conn_01x40, U1 LM1117-3.3, U2 74LVC245A, U3 74LVC245A, U4 74LVC245A, U5 74LVC245A, U6 LISA

Commit message: Redesign of adapter on a 2-layer PCB, changed to 74LVC16244ADGG level shifters, changed sampling clock to C28OUT now sent to the FPGA
Parts:
- removed J1: Conn_01x03, Connector_PinHeader_2.54mm:PinHeader_1x03_P2.54mm_Horizontal, symbol Connector_Generic:Conn_01x03
- removed U2, U3, U4, U5: 74LVC245A, Package_SO:TSSOP-20_4.4x6.5mm_P0.65mm, symbol LISA_to_FPGA:74LVC245A
- added C10, C7, C8, C9: 0.1uF, Capacitor_SMD:C_0603_1608Metric_Pad1.08x0.95mm_HandSolder, symbol Device:C_Small
- added J1: Conn_01x04, Connector_PinHeader_2.54mm:PinHeader_1x04_P2.54mm_Horizontal, symbol Connector_Generic:Conn_01x04
- added U2, U3: 74LVC16244ADGG, Package_SO:TSSOP-48_6.1x12.5mm_P0.5mm, symbol LISA_to_FPGA:74LVC16244ADGG
- R1: value 33 Ω -> 33Ω
- renumbered U6 to U4
Connections:
- net labels added: C28O, C28O_3V3
- net labels removed: C14M_3V3, C14OUT, C14OUT_3V3
- wire segments 38 -> 53
