File: A1200/KiCad/LISA_to_FPGA.sch (KiCad schematic (older format))
At the start: 37 parts, among them J1 Conn_01x01, J2 Conn_01x40, U1 LM1117-3.3, U2 74LVC162244ADGG, U3 74LVC162244ADGG, U4 LISA, U5 RP2354B

Commit message: Add decoupling cap for pin 32 on QFN-80 footprint
Parts:
- added C18: 0.1uF, Capacitor_SMD:C_0603_1608Metric_Pad1.08x0.95mm_HandSolder, symbol Device:C_Small
Connections:
- net 1V1: now also C18.2
- net GND: now also C18.1
Changed lines of the file:
@@
 Connection ~ 5350 7250
-Wire Wire Line
-	5350 7250 6600 7250
 Wire Wire Line
 	5350 7050 5350 6900
@@
 	5350 6900 5050 6900
 Connection ~ 5050 6900
+$Comp
+L Device:C_Small C18
+U 1 1 6B06EF37
+P 2050 7600
+F 0 "C18" H 2142 7646 50  0000 L CNN
+F 1 "0.1uF" H 2100 7750 50  0000 L CNN
+F 2 "Capacitor_SMD:C_0603_1608Metric_Pad1.08x0.95mm_HandSolder" H 2050 7600 50  0001 C CNN
+F 3 "~" H 2050 7600 50  0001 C CNN
+	1    2050 7600
+	1    0    0    -1
+$EndComp
+Wire Wire Line
+	5650 7050 5650 6900
+Wire Wire Line
+	5650 6900 5350 6900
+Connection ~ 5350 6900
+Text GLabel 3100 7700 2    50   Output ~ 0
+1V1
+Wire Wire Line
+	3100 7700 2050 7700
+Wire Wire Line
+	1300 7550 1850 7550
+Wire Wire Line
+	1850 7550 1850 7400
+Wire Wire Line
+	1850 7400 2050 7400
+Connection ~ 1300 7550
+Wire Wire Line
+	2050 7500 2050 7400
+Wire Wire Line
+	5350 7250 6600 7250
+Connection ~ 2050 7400
+Wire Wire Line
+	2050 7400 3100 7400
 $EndSCHEMATC

Commit message: Add decoupling cap for pin 50 on QFN-80 footprint
Parts:
- added C19: 0.1uF, Capacitor_SMD:C_0603_1608Metric_Pad1.08x0.95mm_HandSolder, symbol Device:C_Small
Connections:
- net 3V3: now also C19.2
- net GND: now also C19.1
Changed lines of the file:
@@
 	2050 7500 2050 7400
 Wire Wire Line
-	5350 7250 6600 7250
+	5350 7250 5650 7250
 Connection ~ 2050 7400
 Wire Wire Line
 	2050 7400 3100 7400
+$Comp
+L Device:C_Small C19
+U 1 1 6B09652E
+P 5650 7150
+F 0 "C19" H 5742 7196 50  0000 L CNN
+F 1 "0.1uF" H 5700 7300 50  0000 L CNN
+F 2 "Capacitor_SMD:C_0603_1608Metric_Pad1.08x0.95mm_HandSolder" H 5650 7150 50  0001 C CNN
+F 3 "~" H 5650 7150 50  0001 C CNN
+	1    5650 7150
+	1    0    0    -1
+$EndComp
+Connection ~ 5650 7250
+Wire Wire Line
+	5650 7250 6600 7250
 $EndSCHEMATC
